File: Ear2Ink_PCB_Design/Ear2Ink_PCB_Design.kicad_sch (KiCad schematic)
At the start: 0 parts

Commit message: added some stuff
Other:
- sheet MCU renamed MCU+Mic+UI
- sheet Power Conversions renamed Power Conversions + Battery Monitor
Changed lines of the file:
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@@
 			(color 0 0 0 0.0000)
 		)
-		(property "Sheetname" "MCU"
+		(property "Sheetname" "MCU+Mic+UI"
 			(at 114.3 36.1184 0)
 			(effects
@@
 			(color 0 0 0 0.0000)
 		)
-		(property "Sheetname" "Power Conversions"
+		(property "Sheetname" "Power Conversions + Battery Monitor"
 			(at 31.75 36.1184 0)
 			(effects
