File: Ear2Ink_PCB_Design/mcu.kicad_sch (KiCad schematic)
At the start: 45 parts, among them J1 Conn_01x16_Pin, J2 Conn_01x08_Pin, J3 Conn_01x08_Pin, J4 MEM2052-00-195-00-A_REVA, J5 Conn_01x06_Pin, J6 Conn_01x04_Pin, J7 Conn_01x03_Pin, J8 Conn_01x16_Pin, SW1 SW_Push, U1 STM32F411RETx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

Commit message: Did a lot of stuff
Parts:
- removed J7: Conn_01x03_Pin, Connector_PinHeader_2.54mm:PinHeader_1x03_P2.54mm_Vertical, symbol Connector:Conn_01x03_Pin
- FB1: footprint (none) -> Resistor_SMD:R_0603_1608Metric_Pad0.98x0.95mm_HandSolder
Connections:
- net GND: now also J4.P6 (VSS), J5.1 (Pin_1), R19.2; no longer J5.2 (Pin_2), R19.1
- net SDIO_CMD: now also J5.4 (Pin_4); no longer J5.1 (Pin_1)
- net SD_DAT2: now also J5.2 (Pin_2); no longer J5.4 (Pin_4)
- net at J4.G1 (SHIELD_GND), J4.G2 (SHIELD_GND__1), J4.G3 (SHIELD_GND__2)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: now also R19.1; no longer J4.P6 (VSS), R19.2
Other:
- note added: "DELETED/Replaced with vias"
- moved on the sheet: J5

Commit message: done
Parts:
- added D10, D11, D12, D13, D14, D7, D8, D9: PTVS5V0Z1USK, Diode_SMD:Nexperia_DSN1608-2_1.6x0.8mm, symbol Diode:PTVS5V0Z1USK
Connections:
- net +3.3V: no longer J1.15 (Pin_15), J1.2 (Pin_2), J8.2 (Pin_2), NT2.2, R8.1
- net C1: now also D7.1 (K)
- net C2: now also D8.1 (K)
- net C3: now also D9.1 (K)
- net C4: now also D10.1 (K)
- net GND: now also D10.2 (A), D11.2 (A), D12.2 (A), D13.2 (A), D14.2 (A), D7.2 (A), D8.2 (A), D9.2 (A)
- net R1: now also D11.1 (K)
- net R2: now also D12.1 (K)
- net R3: now also D13.1 (K)
- net R4: now also D14.1 (K)
- new net 5V: J1.15 (Pin_15), J1.2 (Pin_2), J8.2 (Pin_2), NT2.2, R8.1
Other:
- moved on the sheet: C19, D4, J2, J3, J6, R15, SW1
