File: Ear2Ink_PCB_Design/power.kicad_sch (KiCad schematic)
At the start: 31 parts, among them P1 OSTTE020104, U2 TPS562208DDCR, U3 AZ1117-3.3, U5 LM66100DCK, U6 INA213AIDCKR

Commit message: updated 5V resistor values
Parts:
- R1: value 60k -> 54.9k
Changed lines of the file:
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@@
 			)
 		)
-		(property "Value" "60k"
+		(property "Value" "54.9k"
 			(at 198.12 116.8399 0)
 			(effects
